Commit message: RL agent training

File: physical_object/robot_description/xarco/strirus_gamma_body_bridge.xacro (robot description, xacro)
@@ -4,5 +4,5 @@
     <!-- Body description -->
     <link name="base_footprint"/>
-    <joint name="base_footprint_body_1_part_fixed" type="fixed">
+    <joint name="base_footprint_body_1_part_fixed_joint" type="fixed">
         <parent link="base_footprint"/>
         <child link="body_1_part"/>
@@ -38,5 +38,5 @@
     <!-- tof camera 1-->
     <link name="tof_camera_1"></link>
-    <joint name="body_1_part_tof_camera_1_fixed" type="fixed">
+    <joint name="body_1_part_tof_camera_1_fixed_joint" type="fixed">
         <parent link="body_1_part"/>
         <child link="tof_camera_1"/>
@@ -46,5 +46,5 @@
     <!-- imu 1 -->
     <link name="imu_1"></link>
-    <joint name="body_1_part_imu_1_fixed" type="fixed">
+    <joint name="body_1_part_imu_1_fixed_joint" type="fixed">
         <parent link="body_1_part"/>
         <child link="imu_1"/>
@@ -82,5 +82,5 @@
     <!-- tof camera 2 -->
     <link name="tof_camera_2"/>
-    <joint name="body_2_part_tof_camera_2_fixed" type="fixed">
+    <joint name="body_2_part_tof_camera_2_fixed_joint" type="fixed">
         <parent link="body_2_part"/>
         <child link="tof_camera_2"/>
@@ -90,5 +90,5 @@
     <!-- imu 1 -->
     <link name="imu_2"/>
-    <joint name="body_2_part_imu_2_fixed" type="fixed">
+    <joint name="body_2_part_imu_2_fixed_joint" type="fixed">
         <parent link="body_2_part"/>
         <child link="imu_2"/>
@@ -155,5 +155,5 @@
     <xacro:property name="segment_dof" value="${strirus_sim_settings['segments']['segment_dof']}"/>
     <xacro:if value="${str(segment_dof) == '0' or str(segment_dof) == '1up'}">
-        <joint name="segment_side_fixed" type="fixed">
+        <joint name="segment_side_fixed_joint" type="fixed">
             <parent link="body_1_part"/>
             <child link="bridge_1_part"/>
@@ -163,5 +163,5 @@
     </xacro:if>
     <xacro:if value="${str(segment_dof) == '0' or str(segment_dof) == '1side'}">
-        <joint name="segment_up_fixed" type="fixed">
+        <joint name="segment_up_fixed_joint" type="fixed">
             <parent link="bridge_1_part"/>
             <child link="bridge_2_part"/>
@@ -171,5 +171,5 @@
     </xacro:if>
     <xacro:if value="${str(segment_dof) == '1up' or str(segment_dof) == '2'}">
-        <joint name="segment_up_revolute" type="revolute">
+        <joint name="segment_up_revolute_joint" type="revolute">
             <parent link="bridge_1_part"/>
             <child link="bridge_2_part"/>
@@ -186,5 +186,5 @@
     </xacro:if>
     <xacro:if value="${str(segment_dof) == '1side' or str(segment_dof) == '2'}">
-        <joint name="segment_side_revolute" type="revolute">
+        <joint name="segment_side_revolute_joint" type="revolute">
             <parent link="body_1_part"/>
             <child link="bridge_1_part"/>
@@ -200,5 +200,5 @@
         </joint>
     </xacro:if>
-    <joint name="bridge_2_part_body_2_part_fixed" type="fixed">
+    <joint name="bridge_2_part_body_2_part_fixed_joint" type="fixed">
         <parent link="bridge_2_part"/>
         <child link="body_2_part"/>
